File: esp32-ips-display.kicad_pcb (KiCad board)
At the start: 2 copper layers, 50 x 38.5 mm, 25 parts, among them J1 Conn_01x02_Pin, P1 USB_C_Plug_USB2.0, Q1 NPN, Q2 NPN, U1 ESP32-S3-WROOM-1, U2 CH340C, U3 AMS1117-3.3

Commit message: JH
Parts:
- R1: footprint Resistor_SMD:R_0805_2012Metric -> Resistor_SMD:R_0805_2012Metric_Pad1.20x1.40mm_HandSolder
- renumbered R1 to R10
Routing:
- net Net-(J1-Pin_2): track 60.6 -> 0.00 mm, vias 2 -> 0
- net IO0: track 0.00 -> 49.3 mm, vias 0 -> 2
- net MCU_TX0: track 5.00 -> 29.8 mm, vias 1 -> 2
- net MCU_RX0: track 8.42 -> 31.1 mm, vias 1 -> 2
- net MCU_EN: track 73.1 -> 51.3 mm
- net FT0x05_SDA: track 35.9 -> 50.7 mm, vias 2 -> 0
- net Net-(Q2-B): track 14.2 -> 0.00 mm, vias 2 -> 0
- net Net-(Q2-E): track 21.1 -> 32.9 mm, vias 2 -> 0
- net Net-(U4-LEDA): track 56.4 -> 45.2 mm
- net 3v3: track 95.5 -> 106.0 mm, vias 2 -> 3
- net Net-(P1-D-): track 12.1 -> 21.3 mm, vias 2 -> 0
- net VBUS: track 67.6 -> 58.7 mm, vias 0 -> 2
- net Net-(D1-A): track 25.7 -> 34.1 mm
- net FT0x05_SCL: track 34.9 -> 42.0 mm, vias 2 -> 0
- net Net-(U2-V3): track 10.8 -> 6.73 mm
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