File: esp32-ips-display.kicad_sch (KiCad schematic)
At the start: 24 parts, among them J1 Conn_01x02_Pin, P1 USB_C_Plug_USB2.0, Q1 NPN, Q2 NPN, U1 ESP32-S3-WROOM-1, U2 CH340C, U3 AMS1117-3.3

Commit message: JH
Parts:
- R1: footprint Resistor_SMD:R_0805_2012Metric -> Resistor_SMD:R_0805_2012Metric_Pad1.20x1.40mm_HandSolder
Changed lines of the file:
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@@
 			)
 		)
-		(property "Footprint" "Resistor_SMD:R_0805_2012Metric"
+		(property "Footprint" "Resistor_SMD:R_0805_2012Metric_Pad1.20x1.40mm_HandSolder"
 			(at 114.3 163.068 90)
 			(effects
